File: MCU datalogger.kicad_pcb (KiCad board)
At the start: 2 copper layers, 51 x 32.8 mm, 29 parts, among them J1 Conn_01x04_Pin, J2 Conn_01x04_Pin, J3 Conn_01x09_Pin, J4 Conn_02x03_Odd_Even, U1 24LC1025, U2 24LC1025, U3 ATMEGA328P-AU, U4 DS1337S_, Y1 32.768KHz, Y2 16MHz

Commit message: 4 layer
Parts:
- moved U3 0.39 mm to (1965.6, 2098.6)
Routing:
- net /VCC: track 163.4 -> 76.4 mm
- net GND: track 139.0 -> 90.6 mm, vias 9 -> 12
- net Net-(U3-PB7): track 59.3 -> 25.5 mm
- net /MISO: track 57.3 -> 32.1 mm, vias 4 -> 2
- net /SCK: track 97.5 -> 78.6 mm, vias 4 -> 11
- net /MOSI: track 49.3 -> 31.5 mm, vias 0 -> 2
- net /RX: track 27.0 -> 42.2 mm, vias 1 -> 0
- net /RESET: track 23.7 -> 33.6 mm, vias 2 -> 1
- net /TX: track 37.0 -> 43.5 mm, vias 1 -> 0
- net /SDA: track 59.1 -> 62.0 mm, vias 2 -> 5
- net Net-(U3-AREF): track 12.2 -> 13.6 mm
- net Net-(U4-X2): track 7.74 -> 9.06 mm
- net /D2: track 30.2 -> 30.9 mm
- net /D6: track 13.4 -> 14.0 mm
- net Net-(BT1-+): vias 4 -> 3
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- added copper zone on In2.Cu, net /VCC
Other:
- copper layers 2 -> 4
